File: pcb/6ch_old/expansion.brd (EAGLE design)
At the start: 62 x 42 mm, 44 parts, among them IC3 STM32F042F4, J7 AUDIO_JACK_3.5MM_PTH, J8 AUDIO_JACK_3.5MM_PTH, SW3 324_SW, SW4 324_SW, U1 USBC_16P, U2 USBC_16P, U4 XC6206_DEV

Commit message: working on new PCB
Parts:
- removed J7, J8: AUDIO_JACK_3.5MM_PTH, SparkFun-Connectors:AUDIO-JACK
- removed JP9: (no value), pinhead:2X06
- removed LED1, LED2, LED4, LED5, LED6, LED7: (no value), adafruit:CHIP-LED0805
- removed R13, R15, R16, R17, R18, R4: 5K1, joyAnalog:0805
- removed U$14: DG2204R-5.0-8DG2204-8, atx4vc:DG2204R-8
- added J1, J2, J3, J4, J5, J6: AUDIO_JACK_3.5MM_PTH, SparkFun-Connectors:AUDIO-JACK
- added JP1, JP2, JP3, JP4, JP5, JP6: (no value), pinhead:1X03
- added JP7: (no value), adafruit_changed:1X01-CLEANBIG
- added U$1, U$2, U$3, U$4, U$5, U$7: DG2204R-2, expansion:DG2204R-2
- added U$12, U$13: PINHD1X2, adafruit_changed:1X02
- R1, R14, R2, R3, R7: value 5K1 -> 5.1K
- R10, R11, R12, R5, R6, R8, R9: value 5K1 -> 10K
- moved R12 126.0 mm to (81.4, 13.0), turned to 90 degrees
- moved R8 38.0 mm to (45.8, 28.7), turned to 270 degrees
- moved R10 31.6 mm to (30.9, 13.5), turned to 90 degrees
- moved U1 26.5 mm to (84.6, 21.0)
- moved U$10 26.5 mm to (85.5, 3.00)
- moved U$11 26.5 mm to (85.5, 39.0)
- moved LED3 18.6 mm to (29.3, 25.5)
- moved R14 18.1 mm to (25.8, 25.5)
- moved R11 18.1 mm to (56.0, 13.5), turned to 90 degrees
- moved C3 18.0 mm to (18.7, 24.3), turned to 90 degrees
- moved R9 17.6 mm to (71.0, 28.7), turned to 270 degrees
- moved C2 17.1 mm to (32.4, 21.8)
- moved IC3 14.5 mm to (38.1, 21.1)
- moved R6 14.3 mm to (20.7, 28.8), turned to 270 degrees
- moved U4 13.2 mm to (15.0, 24.3), turned to 90 degrees
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Connections:
- removed net CH_PA0: IC3.6, LED5.C, R9.1, U$14.P$10, U$14.P$9
- removed net CH_PA1: IC3.7, LED4.C, R8.1, U$14.P$7, U$14.P$8
- removed net CH_PA4: IC3.10, LED2.C, R6.1, U$14.P$5, U$14.P$6
- removed net CH_PA5: IC3.11
- removed net CH_PB1: IC3.14, LED1.C, R4.1, U$14.P$3, U$14.P$4
- removed net CH_PF0: IC3.2, LED7.C, R11.1, U$14.P$13, U$14.P$14
- removed net CH_PF1: IC3.3, LED6.C, R10.1, U$14.P$11, U$14.P$12
- removed net N$3: LED1.A, R12.2
- removed net N$4: LED2.A, R13.2
- removed net N$5: LED4.A, R15.2
- removed net N$6: LED5.A, R16.2
- removed net N$7: LED6.A, R17.2
- removed net N$8: LED7.A, R18.2
- new net CH1: IC3.6, J1.TIP, JP1.2, R6.1, U$4.P$3, U$4.P$4
- new net CH2: IC3.7, J5.TIP, JP2.2, R8.1, U$5.P$3, U$5.P$4
- new net CH3: IC3.10, J6.TIP, JP3.2, R9.1, U$7.P$3, U$7.P$4
- new net CH4: IC3.14, J4.TIP, JP4.2, R10.1, U$1.P$1, U$1.P$2
- new net CH5: IC3.2, J2.TIP, JP5.2, R11.1, U$2.P$1, U$2.P$2
- new net CH6: IC3.3, J3.TIP, JP6.2, R12.1, U$3.P$1, U$3.P$2
- new net N$13: IC3.11, J1.RING, JP7.1
- net +3V3: now also JP1.1, JP2.1, JP3.1, JP4.1, JP5.1, JP6.1, R12.2; no longer R12.1, R13.1, R15.1, R16.1, R17.1, R18.1, R4.2
- net GND: now also J1.SLEEVE, J2.SLEEVE, J3.SLEEVE, J4.SLEEVE, J5.SLEEVE, J6.SLEEVE, JP1.3, JP2.3, JP3.3, JP4.3, JP5.3, JP6.3, U$1.P$3, U$1.P$4, U$2.P$3, U$2.P$4, U$3.P$3, U$3.P$4, U$4.P$1, U$4.P$2, U$5.P$1, U$5.P$2, U$7.P$1, U$7.P$2; no longer U$14.P$1, U$14.P$15, U$14.P$16, U$14.P$2
- net U2RX: now also U$13.1
- net U2TX: now also U$13.2
- net USBDN/U1TX: now also U$12.2
- net USBDP/U1RX: now also U$12.1
Routing:
- net +3V3: track 0.00 -> 222.6 mm
- net CH4: track 0.00 -> 110.8 mm
- net +5V: track 0.00 -> 93.7 mm, vias 0 -> 4
- net U2RX: track 0.00 -> 64.0 mm
- net CH6: track 0.00 -> 63.0 mm
- net CH3: track 0.00 -> 61.9 mm
- net N$14: track 0.00 -> 54.2 mm, vias 0 -> 1
- net CH1: track 0.00 -> 47.5 mm
- net U2TX: track 0.00 -> 47.1 mm
- net CH2: track 0.00 -> 41.0 mm
- net CH5: track 0.00 -> 38.2 mm
- net USBDN/U1TX: track 0.00 -> 31.1 mm
- net USBDP/U1RX: track 0.00 -> 30.7 mm
- net N$13: track 0.00 -> 23.7 mm, vias 0 -> 1
- net BUTTON1: track 0.00 -> 22.2 mm
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Other:
- board size 62 x 42 mm -> 88 x 42 mm
- board text added: "0"
- board text added: "3V"
- board text added: "S1"
- board text added: "S2"
- board text added: "S3"
- board text added: "S4"
- board text added: "S5"
- board text removed: "6"
- board text removed: "GND"
