File: pcb/6ch_old/expansion.sch (EAGLE design)
At the start: 44 parts, among them IC3 STM32F042F4, J7 AUDIO_JACK_3.5MM_PTH, J8 AUDIO_JACK_3.5MM_PTH, SW3 324_SW, SW4 324_SW, U1 USBC_16P, U2 USBC_16P, U4 XC6206_DEV

Commit message: working on new PCB
Parts:
- removed J7, J8: AUDIO_JACK_3.5MM_PTH, SparkFun-Connectors:AUDIO_JACK_3.5MM_PTH
- removed JP9: (no value), pinhead:PINHD-2X6
- removed LED1, LED2, LED4, LED5, LED6, LED7: (no value), adafruit:LEDCHIP-LED0805
- removed R13, R15, R16, R17, R18, R4: 5K1, joyAnalog:RESISTOR0805-RES
- removed U$14: DG2204R-5.0-8DG2204-8, atx4vc:DG2204R-5.0-8DG2204-8
- added J1, J2, J3, J4, J5, J6: AUDIO_JACK_3.5MM_PTH, SparkFun-Connectors:AUDIO_JACK_3.5MM_PTH
- added JP1, JP2, JP3, JP4, JP5, JP6: (no value), pinhead:PINHD-1X3
- added JP7: (no value), adafruit_changed:PINHD-1X1CB
- added U$1, U$2, U$3, U$4, U$5, U$7: DG2204R-2, expansion:DG2204R-2
- added U$12, U$13: PINHD1X2, adafruit_changed:PINHD1X2
- R1, R14, R2, R3, R7: value 5K1 -> 5.1K
- R10, R11, R12, R5, R6, R8, R9: value 5K1 -> 10K
Connections:
- removed net CH_PA0: IC3.PA0, LED5.C, R9.1, U$14.P$5
- removed net CH_PA1: IC3.PA1, LED4.C, R8.1, U$14.P$4
- removed net CH_PA4: IC3.PA4, LED2.C, R6.1, U$14.P$3
- removed net CH_PA5: IC3.PA5
- removed net CH_PB1: IC3.PB1, LED1.C, R4.1, U$14.P$2
- removed net CH_PF0: IC3.PF0/OSC_IN, LED7.C, R11.1, U$14.P$7
- removed net CH_PF1: IC3.PF1/OSC_OUT, LED6.C, R10.1, U$14.P$6
- removed net N$3: LED1.A, R12.2
- removed net N$4: LED2.A, R13.2
- removed net N$5: LED4.A, R15.2
- removed net N$6: LED5.A, R16.2
- removed net N$7: LED6.A, R17.2
- removed net N$8: LED7.A, R18.2
- new net CH1: IC3.PA0, J1.TIP, JP1.2, R6.1, U$4.P$2
- new net CH2: IC3.PA1, J5.TIP, JP2.2, R8.1, U$5.P$2
- new net CH3: IC3.PA4, J6.TIP, JP3.2, R9.1, U$7.P$2
- new net CH4: IC3.PB1, J4.TIP, JP4.2, R10.1, U$1.P$1
- new net CH5: IC3.PF0/OSC_IN, J2.TIP, JP5.2, R11.1, U$2.P$1
- new net CH6: IC3.PF1/OSC_OUT, J3.TIP, JP6.2, R12.1, U$3.P$1
- new net N$13: IC3.PA5, J1.RING, JP7.1
- net +3V3: now also JP1.1, JP2.1, JP3.1, JP4.1, JP5.1, JP6.1, R12.2; no longer R12.1, R13.1, R15.1, R16.1, R17.1, R18.1, R4.2
- net GND: now also J1.SLEEVE, J2.SLEEVE, J3.SLEEVE, J4.SLEEVE, J5.SLEEVE, J6.SLEEVE, JP1.3, JP2.3, JP3.3, JP4.3, JP5.3, JP6.3, U$1.P$2, U$2.P$2, U$3.P$2, U$4.P$1, U$5.P$1, U$7.P$1; no longer U$14.P$1, U$14.P$8
- net U2RX: now also U$13.1
- net U2TX: now also U$13.2
- net USBDN/U1TX: now also U$12.2
- net USBDP/U1RX: now also U$12.1
Other:
- moved on the sheet: R10, R11, R12, R6, R8, R9
