File: pcb/6ch/expansion.sch (EAGLE design)
At the start: 44 parts, among them IC3 STM32F042F4, J7 AUDIO_JACK_3.5MM_PTH, J8 AUDIO_JACK_3.5MM_PTH, SW3 324_SW, SW4 324_SW, U1 USBC_16P, U2 USBC_16P, U4 XC6206_DEV

Commit message: working on new PCB
Connections:
- net CH_PA0: now also JP9.8
- net CH_PA1: now also JP9.10, LED6.C, R10.1, U$14.P$6; no longer LED4.C, R8.1, U$14.P$4
- net CH_PA4: now also JP9.12, LED7.C, R11.1, U$14.P$7; no longer LED2.C, R6.1, U$14.P$3
- net CH_PA5: now also JP9.2, LED1.C, R4.1, U$14.P$2
- net CH_PB1: no longer LED1.C, R4.1, U$14.P$2
- net CH_PF0: now also JP9.4, LED2.C, R6.1, U$14.P$3; no longer LED7.C, R11.1, U$14.P$7
- net CH_PF1: now also JP9.6, LED4.C, R8.1, U$14.P$4; no longer LED6.C, R10.1, U$14.P$6
- net GND: now also JP9.1, JP9.11, JP9.3, JP9.5, JP9.7, JP9.9
Other:
- moved on the sheet: JP9

Commit message: working on new PCB
Parts:
- added JP1: (no value), adafruit_changed:PINHD-1X1CB
- added JP2: (no value), pinhead:PINHD-2X3
- added U$1, U$3: PINHD1X2, adafruit_changed:PINHD1X2
Connections:
- net +3V3: now also JP2.5, JP2.6, U$6.5; no longer U$6.1
- net +5V: now also JP2.1, JP2.2
- net CH_PA4: now also J8.TIP
- net CH_PA5: now also J7.TIP
- net CH_PB1: now also J7.RING, JP1.1
- net GND: now also J7.SLEEVE, J8.SLEEVE, JP2.3, JP2.4, U$6.1; no longer U$6.5
- net U2RX: now also U$1.2
- net U2TX: now also U$1.1
- net USBDN/U1TX: now also U$3.1
- net USBDP/U1RX: now also U$3.2
Other:
- moved on the sheet: J7, J8
