File: pcb/6ch/expansion.sch (EAGLE design)
At the start: 55 parts, among them IC3 STM32F042F4, J7 AUDIO_JACK_3.5MM_PTH, J8 AUDIO_JACK_3.5MM_PTH, SW3 324_SW, SW4 324_SW, U1 USBC_16P, U2 USBC_16P, U4 XC6206_DEV

Commit message: moved channel 7 to terminal and on header
Parts:
- removed U$4: PINHD1X2, adafruit_changed:PINHD1X2
- added JP1, JP3: (no value), pinhead:PINHD-1X1
Connections:
- net CH_PA6: now also U$2.1; no longer U$4.2
- net CH_PB1: now also JP1.1, U$14.P$1; no longer U$2.2
- net GND: now also JP3.1, U$2.2; no longer U$14.P$1, U$2.1, U$4.1
Other:
- moved on the sheet: U$2
Changed lines of the file:
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@@
 <part name="J8" library="SparkFun-Connectors" deviceset="AUDIO_JACK_3.5MM" device="_PTH"/>
 <part name="JP9" library="pinhead" library_urn="urn:adsk.eagle:library:325" deviceset="PINHD-2X6" device="" package3d_urn="urn:adsk.eagle:package:22474/2"/>
-<part name="GND9" library="supply1" deviceset="GND" device=""/>
 <part name="GND13" library="supply1" deviceset="GND" device=""/>
 <part name="R4" library="joyAnalog" deviceset="RESISTOR" device="0805-RES" value="5K1"/>
@@
 <part name="R20" library="joyAnalog" deviceset="RESISTOR" device="0805-RES" value="5K1"/>
 <part name="+3V21" library="supply1" library_urn="urn:adsk.eagle:library:371" deviceset="+3V3" device=""/>
-<part name="U$2" library="adafruit_changed" deviceset="PINHD1X2" device=""/>
-<part name="GND21" library="supply1" deviceset="GND" device=""/>
 <part name="R21" library="joyAnalog" deviceset="RESISTOR" device="0805-RES" value="5K1"/>
 <part name="+3V22" library="supply1" library_urn="urn:adsk.eagle:library:371" deviceset="+3V3" device=""/>
@@
 <part name="R22" library="joyAnalog" deviceset="RESISTOR" device="0805-RES" value="5K1"/>
 <part name="+3V23" library="supply1" library_urn="urn:adsk.eagle:library:371" deviceset="+3V3" device=""/>
-<part name="U$4" library="adafruit_changed" deviceset="PINHD1X2" device=""/>
-<part name="GND22" library="supply1" deviceset="GND" device=""/>
+<part name="JP1" library="pinhead" library_urn="urn:adsk.eagle:library:325" deviceset="PINHD-1X1" device="" package3d_urn="urn:adsk.eagle:package:22485/2"/>
+<part name="JP3" library="pinhead" library_urn="urn:adsk.eagle:library:325" deviceset="PINHD-1X1" device="" package3d_urn="urn:adsk.eagle:package:22485/2"/>
+<part name="GND23" library="supply1" deviceset="GND" device=""/>
+<part name="U$2" library="adafruit_changed" deviceset="PINHD1X2" device=""/>
+<part name="GND21" library="supply1" deviceset="GND" device=""/>
 </parts>
 <sheets>
@@
 <attribute name="VALUE" x="-265.43" y="-76.2" size="1.778" layer="96"/>
 </instance>
-<instance part="GND9" gate="1" x="-208.28" y="-55.88" smashed="yes" rot="MR0">
-<attribute name="VALUE" x="-205.74" y="-58.42" size="1.778" layer="96" rot="MR0"/>
-</instance>
 <instance part="GND13" gate="1" x="-208.28" y="-91.44" smashed="yes" rot="MR0">
 <attribute name="VALUE" x="-205.74" y="-93.98" size="1.778" layer="96" rot="MR0"/>
@@
 <attribute name="VALUE" x="-119.38" y="-121.92" size="1.778" layer="96" rot="MR90"/>
 </instance>
-<instance part="U$2" gate="1" x="-147.32" y="-142.24" smashed="yes" rot="R180">
-<attribute name="NAME" x="-140.97" y="-147.955" size="1.778" layer="95" rot="R180"/>
-<attribute name="VALUE" x="-140.97" y="-137.16" size="1.778" layer="96" rot="R180"/>
-</instance>
-<instance part="GND21" gate="1" x="-134.62" y="-147.32" smashed="yes" rot="MR0">
-<attribute name="VALUE" x="-132.08" y="-149.86" size="1.778" layer="96" rot="MR0"/>
-</instance>
 <instance part="R21" gate="G$1" x="-48.26" y="-124.46" smashed="yes" rot="MR90">
 <attribute name="NAME" x="-46.7614" y="-128.27" size="1.778" layer="95" rot="MR90"/>
@@
 <attribute name="VALUE" x="-58.42" y="-109.22" size="1.778" layer="96" rot="MR90"/>
 </instance>
-<instance part="U$4" gate="1" x="-71.12" y="-139.7" smashed="yes" rot="R180">
-<attribute name="NAME" x="-64.77" y="-145.415" size="1.778" layer="95" rot="R180"/>
-<attribute name="VALUE" x="-64.77" y="-134.62" size="1.778" layer="96" rot="R180"/>
-</instance>
-<instance part="GND22" gate="1" x="-68.58" y="-152.4" smashed="yes" rot="MR0">
-<attribute name="VALUE" x="-66.04" y="-154.94" size="1.778" layer="96" rot="MR0"/>
+<instance part="JP1" gate="G$1" x="-147.32" y="-142.24" smashed="yes" rot="R180">
+<attribute name="NAME" x="-151.13" y="-142.875" size="1.778" layer="95" rot="R180"/>
+<attribute name="VALUE" x="-140.97" y="-137.16" size="1.778" layer="96" rot="R180"/>
+</instance>
+<instance part="JP3" gate="G$1" x="-172.72" y="-157.48" smashed="yes" rot="R180">
+<attribute name="NAME" x="-166.37" y="-160.655" size="1.778" layer="95" rot="R180"/>
+<attribute name="VALUE" x="-166.37" y="-152.4" size="1.778" layer="96" rot="R180"/>
+</instance>
+<instance part="GND23" gate="1" x="-160.02" y="-162.56" smashed="yes" rot="MR0">
+<attribute name="VALUE" x="-157.48" y="-165.1" size="1.778" layer="96" rot="MR0"/>
+</instance>
+<instance part="U$2" gate="1" x="-66.04" y="-137.16" smashed="yes">
+<attribute name="NAME" x="-72.39" y="-131.445" size="1.778" layer="95"/>
+<attribute name="VALUE" x="-72.39" y="-142.24" size="1.778" layer="96"/>
+</instance>
+<instance part="GND21" gate="1" x="-78.74" y="-139.7" smashed="yes" rot="MR0">
+<attribute name="VALUE" x="-76.2" y="-142.24" size="1.778" layer="96" rot="MR0"/>
 </instance>
 </instances>
@@
 <pinref part="GND13" gate="1" pin="GND"/>
 <wire x1="-185.42" y1="-88.9" x2="-208.28" y2="-88.9" width="0.1524" layer="91"/>
-</segment>
-<segment>
-<pinref part="U$14" gate="G$1" pin="P$1"/>
-<pinref part="GND9" gate="1" pin="GND"/>
-<wire x1="-185.42" y1="-53.34" x2="-208.28" y2="-53.34" width="0.1524" layer="91"/>
 </segment>
 <segment>
@@
 </segment>
 <segment>
-<pinref part="U$2" gate="1" pin="1"/>
+<pinref part="JP3" gate="G$1" pin="1"/>
+<pinref part="GND23" gate="1" pin="GND"/>
+<wire x1="-170.18" y1="-157.48" x2="-160.02" y2="-157.48" width="0.1524" layer="91"/>
+<wire x1="-160.02" y1="-157.48" x2="-160.02" y2="-160.02" width="0.1524" layer="91"/>
+</segment>
+<segment>
+<pinref part="U$2" gate="1" pin="2"/>
 <pinref part="GND21" gate="1" pin="GND"/>
-<wire x1="-144.78" y1="-144.78" x2="-134.62" y2="-144.78" width="0.1524" layer="91"/>
-</segment>
-<segment>
-<pinref part="U$4" gate="1" pin="1"/>
-<pinref part="GND22" gate="1" pin="GND"/>
-<wire x1="-68.58" y1="-142.24" x2="-68.58" y2="-149.86" width="0.1524" layer="91"/>
+<wire x1="-68.58" y1="-137.16" x2="-78.74" y2="-137.16" width="0.1524" layer="91"/>
 </segment>
 </net>
@@
 <pinref part="LED8" gate="G$1" pin="C"/>
 <junction x="-121.92" y="-142.24"/>
-<pinref part="U$2" gate="1" pin="2"/>
 <wire x1="-134.62" y1="-142.24" x2="-144.78" y2="-142.24" width="0.1524" layer="91"/>
 <junction x="-134.62" y="-142.24"/>
+<pinref part="JP1" gate="G$1" pin="1"/>
+</segment>
+<segment>
+<wire x1="-172.72" y1="-53.34" x2="-185.42" y2="-53.34" width="0.1524" layer="91"/>
+<pinref part="U$14" gate="G$1" pin="P$1"/>
+<label x="-180.34" y="-53.34" size="1.778" layer="95"/>
 </segment>
 </net>
@@
 <wire x1="-96.52" y1="-106.68" x2="-96.52" y2="-129.54" width="0.1524" layer="91"/>
 <label x="-35.56" y="-129.54" size="1.778" layer="95"/>
-<wire x1="-96.52" y1="-129.54" x2="-68.58" y2="-129.54" width="0.1524" layer="91"/>
+<wire x1="-96.52" y1="-129.54" x2="-78.74" y2="-129.54" width="0.1524" layer="91"/>
 <pinref part="R21" gate="G$1" pin="1"/>
-<wire x1="-68.58" y1="-129.54" x2="-60.96" y2="-129.54" width="0.1524" layer="91"/>
+<wire x1="-78.74" y1="-129.54" x2="-60.96" y2="-129.54" width="0.1524" layer="91"/>
 <wire x1="-60.96" y1="-129.54" x2="-48.26" y2="-129.54" width="0.1524" layer="91"/>
 <wire x1="-48.26" y1="-129.54" x2="-25.4" y2="-129.54" width="0.1524" layer="91"/>
@@
 <pinref part="LED9" gate="G$1" pin="C"/>
 <junction x="-60.96" y="-129.54"/>
-<pinref part="U$4" gate="1" pin="2"/>
-<wire x1="-68.58" y1="-129.54" x2="-68.58" y2="-139.7" width="0.1524" layer="91"/>
-<junction x="-68.58" y="-129.54"/>
-</segment>
-</net>
+<pinref part="U$2" gate="1" pin="1"/>
+<wire x1="-68.58" y1="-134.62" x2="-78.74" y2="-134.62" width="0.1524" layer="91"/>
+<wire x1="-78.74" y1="-134.62" x2="-78.74" y2="-129.54" width="0.1524" layer="91"/>
+<junction x="-78.74" y="-129.54"/>
+</segment>
+</net>
