File: pcb/6ch/expansion.brd (EAGLE design)
At the start: 62 x 42 mm, 44 parts, among them IC3 STM32F042F4, J7 AUDIO_JACK_3.5MM_PTH, J8 AUDIO_JACK_3.5MM_PTH, SW3 324_SW, SW4 324_SW, U1 USBC_16P, U2 USBC_16P, U4 XC6206_DEV

Commit message: working on new PCB
Parts:
- moved R18 120.1 mm to (43.7, 19.1)
- moved LED7 117.6 mm to (43.7, 21.2), turned to 90 degrees
- moved R17 110.4 mm to (38.7, 19.1)
- moved LED6 107.9 mm to (38.7, 21.2), turned to 90 degrees
- moved R16 100.7 mm to (33.8, 19.1)
- moved LED5 98.1 mm to (33.8, 21.2), turned to 90 degrees
- moved R15 91.2 mm to (28.7, 19.1), turned to 180 degrees
- moved LED4 88.9 mm to (28.7, 21.2), turned to 270 degrees
- moved R13 82.1 mm to (23.7, 19.1), turned to 180 degrees
- moved LED2 79.9 mm to (23.6, 21.2), turned to 270 degrees
- moved LED1 72.4 mm to (18.8, 21.2), turned to 270 degrees
- moved R12 67.8 mm to (18.8, 19.1), turned to 180 degrees
- moved JP9 65.8 mm to (31.0, 14.5)
- moved R3 32.6 mm to (51.3, 15.6)
- moved R7 29.2 mm to (54.5, 28.8), turned to 0 degrees
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Connections:
- net CH_PA0: now also JP9.8
- net CH_PA1: now also JP9.10, LED6.C, R10.1, U$14.P$11, U$14.P$12; no longer LED4.C, R8.1, U$14.P$7, U$14.P$8
- net CH_PA4: now also JP9.12, LED7.C, R11.1, U$14.P$13, U$14.P$14; no longer LED2.C, R6.1, U$14.P$5, U$14.P$6
- net CH_PA5: now also JP9.2, LED1.C, R4.1, U$14.P$3, U$14.P$4
- net CH_PB1: no longer LED1.C, R4.1, U$14.P$3, U$14.P$4
- net CH_PF0: now also JP9.4, LED2.C, R6.1, U$14.P$5, U$14.P$6; no longer LED7.C, R11.1, U$14.P$13, U$14.P$14
- net CH_PF1: now also JP9.6, LED4.C, R8.1, U$14.P$7, U$14.P$8; no longer LED6.C, R10.1, U$14.P$11, U$14.P$12
- net GND: now also JP9.1, JP9.11, JP9.3, JP9.5, JP9.7, JP9.9
Routing:
- net CH_PF1: track 0.00 -> 53.6 mm
- net CH_PA0: track 0.00 -> 50.2 mm
- net CH_PF0: track 0.00 -> 50.0 mm
- net CH_PA1: track 0.00 -> 46.9 mm
- net U2TX: track 0.00 -> 43.7 mm
- net CH_PA4: track 0.00 -> 40.7 mm
- net CH_PA5: track 0.00 -> 40.5 mm
- net USBDN/U1TX: track 0.00 -> 34.4 mm
- net USBDP/U1RX: track 0.00 -> 33.7 mm
- net +3V3: track 0.00 -> 30.8 mm, vias 0 -> 8
- net U2RX: track 0.00 -> 28.8 mm
- net +5V: track 0.00 -> 19.2 mm
- net BUTTON1: track 0.00 -> 10.1 mm
- net N$14: track 0.00 -> 9.53 mm
- net N$31: track 0.00 -> 9.13 mm
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
Commit message: working on new PCB
Parts:
- added JP1: (no value), adafruit_changed:1X01-CLEANBIG
- added JP2: (no value), pinhead:2X03
- added U$1, U$3: PINHD1X2, adafruit_changed:1X02
- moved C2 0.51 mm to (24.9, 8.13)
- moved U$6 0.38 mm to (29.0, 1.65)
- moved C4 0.13 mm to (37.0, 7.62)
- turned R7 to 180 degrees
Connections:
- net +3V3: now also JP2.5, JP2.6, U$6.5; no longer U$6.1
- net +5V: now also JP2.1, JP2.2
- net CH_PA4: now also J8.TIP
- net CH_PA5: now also J7.TIP
- net CH_PB1: now also J7.RING, JP1.1
- net GND: now also J7.SLEEVE, J8.SLEEVE, JP2.3, JP2.4, U$6.1; no longer U$6.5
- net U2RX: now also U$1.2
- net U2TX: now also U$1.1
- net USBDN/U1TX: now also U$3.1
- net USBDP/U1RX: now also U$3.2
Routing:
- net +3V3: track 30.8 -> 217.9 mm, vias 8 -> 11
- net GND: track 0.00 -> 99.1 mm
- net +5V: track 19.2 -> 87.9 mm, vias 0 -> 3
- net CH_PB1: track 0.00 -> 26.8 mm, vias 0 -> 1
- net CH_PA4: track 40.7 -> 61.3 mm
- net CH_PA5: track 40.5 -> 50.5 mm
- net USBDN/U1TX: track 34.4 -> 32.3 mm
- net N$11: track 0.00 -> 1.84 mm
- net USBDP/U1RX: track 33.7 -> 32.2 mm
- net N$2: track 6.76 -> 8.30 mm
- net U2TX: track 43.7 -> 44.6 mm
- net N$1: track 6.24 -> 7.00 mm
- net SWDIO: track 5.58 -> 4.89 mm
Other:
- board text added: "5V"
- board text added: "U2R"
- board text added: "U2T"
- board text added: "dekuNukem 2024"
- board text added: "duckyPad Pro Expansion Module"
- board text added: "duckyPad.com"
- board text removed: "U1R"
- board text removed: "U1T"
- board text removed: "U2RX"
- board text removed: "U2TX"
- board text removed: "duckyPad Pro Expansion Module dekuNukem 2024"

Commit message: working on new PCB
Parts:
- moved LED3 4.15 mm to (23.6, 10.7), turned to 90 degrees
- moved R14 2.37 mm to (20.8, 12.2), turned to 270 degrees
- moved U$1 2.16 mm to (45.6, 15.9)
Routing:
- net N$12: track 8.63 -> 4.65 mm
- net +3V3: track 217.9 -> 219.1 mm
Other:
- outline, holes or cut-outs redrawn
- board text added: "PB1"
- board text removed: "PC"
